File: circuts/kotel.kicad_pcb (KiCad board)
At the start: 2 copper layers, 21 parts, among them IC1 ATMEGA328P-TQFP32, P1 Power, P2 RELE CONNECTOR, P3 UART_RST, P4 TWI SW, Q1 MOS_N, U1 MAX6634, U2 7805, X1 12mHz

Commit message: Fixed software SDL/SCL.
Parts:
- moved U1 4.64 mm to (204.6, 164.4)
- moved R1 2.15 mm to (191.6, 162.6)
- moved R3 1.28 mm to (186.0, 162.6)
Connections:
- IC1 pad 23: /SDA SW -> /SDL SW
- IC1 pad 24: /SDL SW -> /SDA SW
- P4 pad 2: /SDL SW -> /SDA SW
- P4 pad 3: /SDA SW -> /SDL SW
- R1 pad 1: /SDL SW -> /SDA SW
- R3 pad 1: /SDA SW -> /SDL SW
Routing:
- net /SDL: track 39.2 -> 44.8 mm
- net GND: track 168.4 -> 173.8 mm
- net /!ALERT: track 10.7 -> 15.4 mm
- net /SDA: track 14.3 -> 18.3 mm
- net +5V: track 161.2 -> 162.8 mm
- net /SDA SW: track 8.04 -> 6.54 mm
- net /SDL SW: track 8.91 -> 8.39 mm
Other:
- board text added: "Created by ASM. Kotel v.0.2 2013"
- board text removed: "Created by ASM. Kotel v.0.1 2013"
